File: Ahoura_Blinky.brd (EAGLE design)
At the start: 21.3 x 30.5 mm, 13 parts

Commit message: more updates
Parts:
- C2, C3: value (none) -> 100n
- R3: value (none) -> 10k
Connections:
- removed net N$10: R4.2, R5.2
- removed net N$11: OP1.7, R6.1
- new net N$3: OP1.7, R4.2, R5.2, R6.1
Routing:
- net N$10: track 13.9 -> 0.00 mm, vias 2 -> 0
- net N$3: track 0.00 -> 13.8 mm, vias 0 -> 2
- net N$11: track 3.41 -> 0.00 mm
- net N$4: track 15.3 -> 14.7 mm
Other:
- board text added: "ON"
