File: Ahoura_Blinky.sch (EAGLE design)
At the start: 13 parts

Commit message: more updates
Parts:
- C2, C3: value (none) -> 100n
- R3: value (none) -> 10k
Connections:
- removed net N$10: R4.2, R5.2
- removed net N$11: OP1B.OUT, R6.1
- new net N$3: OP1B.OUT, R4.2, R5.2, R6.1
Changed lines of the file:
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@@
 <part name="R1" library="CalvEngIO-Passives" deviceset="RESISTOR" device="0402"/>
 <part name="R2" library="CalvEngIO-Passives" deviceset="RESISTOR" device="0402"/>
-<part name="R3" library="CalvEngIO-Passives" deviceset="RESISTOR" device="0402"/>
+<part name="R3" library="CalvEngIO-Passives" deviceset="RESISTOR" device="0402" value="10k"/>
 <part name="R4" library="CalvEngIO-Passives" deviceset="RESISTOR" device="0402"/>
 <part name="R5" library="CalvEngIO-Passives" deviceset="RESISTOR" device="0402"/>
 <part name="R6" library="CalvEngIO-Passives" deviceset="RESISTOR" device="0402"/>
 <part name="C1" library="CalvEngIO-Passives" deviceset="CAPACITOR" device="0402"/>
-<part name="C2" library="CalvEngIO-Passives" deviceset="CAPACITOR" device="0402"/>
+<part name="C2" library="CalvEngIO-Passives" deviceset="CAPACITOR" device="0402" value="100n"/>
 <part name="OP1" library="CalvEngIO-AnalogIC" deviceset="OP-DUAL" device="RM"/>
 <part name="LED1" library="CalvEngIO-LED" deviceset="LED" device="0603"/>
-<part name="SUPPLY1" library="CalvEngIO-Symbols" deviceset="3.3V" device=""/>
 <part name="SUPPLY2" library="CalvEngIO-Symbols" deviceset="3.3V" device=""/>
 <part name="SUPPLY4" library="CalvEngIO-Symbols" deviceset="3.3V" device=""/>
@@
 <part name="GND3" library="CalvEngIO-Symbols" deviceset="GND" device=""/>
 <part name="GND4" library="CalvEngIO-Symbols" deviceset="GND" device=""/>
-<part name="C3" library="CalvEngIO-Passives" deviceset="CAPACITOR" device="0402"/>
+<part name="C3" library="CalvEngIO-Passives" deviceset="CAPACITOR" device="0402" value="100n"/>
 <part name="GND5" library="CalvEngIO-Symbols" deviceset="GND" device=""/>
 </parts>
@@
 <instance part="OP1" gate="B" x="101.6" y="66.04"/>
 <instance part="LED1" gate="G$1" x="129.54" y="55.88"/>
-<instance part="SUPPLY1" gate="G$1" x="73.66" y="40.64"/>
 <instance part="SUPPLY2" gate="G$1" x="30.48" y="60.96"/>
 <instance part="SUPPLY4" gate="G$1" x="53.34" y="55.88"/>
@@
 </segment>
 </net>
-<net name="N$10" class="0">
-<segment>
-<pinref part="R5" gate="G$1" pin="2"/>
-<wire x1="106.68" y1="55.88" x2="111.76" y2="55.88" width="0.1524" layer="91"/>
-<wire x1="111.76" y1="55.88" x2="111.76" y2="78.74" width="0.1524" layer="91"/>
-<pinref part="R4" gate="G$1" pin="2"/>
-<wire x1="111.76" y1="78.74" x2="99.06" y2="78.74" width="0.1524" layer="91"/>
-</segment>
-</net>
-<net name="N$11" class="0">
-<segment>
-<pinref part="OP1" gate="B" pin="OUT"/>
-<pinref part="R6" gate="G$1" pin="1"/>
-<wire x1="109.22" y1="66.04" x2="114.3" y2="66.04" width="0.1524" layer="91"/>
-</segment>
-</net>
 <net name="N$12" class="0">
 <segment>
@@
 </segment>
 </net>
+<net name="N$3" class="0">
+<segment>
+<pinref part="R5" gate="G$1" pin="2"/>
+<wire x1="106.68" y1="55.88" x2="111.76" y2="55.88" width="0.1524" layer="91"/>
+<pinref part="R4" gate="G$1" pin="2"/>
+<wire x1="111.76" y1="78.74" x2="99.06" y2="78.74" width="0.1524" layer="91"/>
+<wire x1="111.76" y1="78.74" x2="111.76" y2="66.04" width="0.1524" layer="91"/>
+<pinref part="OP1" gate="B" pin="OUT"/>
+<wire x1="111.76" y1="66.04" x2="109.22" y2="66.04" width="0.1524" layer="91"/>
+<wire x1="111.76" y1="55.88" x2="111.76" y2="66.04" width="0.1524" layer="91"/>
+<junction x="111.76" y="66.04"/>
+<pinref part="R6" gate="G$1" pin="1"/>
+<wire x1="114.3" y1="66.04" x2="111.76" y2="66.04" width="0.1524" layer="91"/>
+</segment>
+</net>
